Commit message: agrega codigos modulo2

File: modulo2/src/ros2_ws/src/my_robot_description/urdf/mobile_base.xacro (robot description, xacro)
@@ -10,7 +10,7 @@
         <visual>
             <geometry>
-                <box size="${base_length} ${base_width} ${base_height}" />
+                <mesh filename="package://my_robot_description/meshes/base_link.STL" scale="1.0"/>
             </geometry>
-            <origin xyz="0 0 ${base_height / 2.0}" rpy="0 0 0" />
+            <origin xyz="0 0 0.1" rpy="0 0 0" />
             <material name="blue" />
         </visual>

File: modulo2/src/ros2_ws/src/my_robot_description/urdf/my_robot.urdf (robot description, URDF)
Before this commit: robot my_robot, 5 links, 4 joints
Links:
- link base_link: geometry visual mesh filename=package://my_robot_description/meshes/base_link.STL scale=1.0 1.0 1.0
